File: KiCAD_files/Morpheus_PPG_RevA1.sch (KiCad schematic (older format))
At the start: 38 parts, among them P1 CONN_01X01, P10 CONN_01X04, P11 CONN_01X03, P12 CONN_01X04, P2 CONN_01X01, P3 CONN_01X01, P4 CONN_01X01, P5 CONN_01X01, P6 CONN_01X04, P7 CONN_01X04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

Commit message: Corrected DNCs, RESET_N, and simplified traces
Less cluttered now. All 130 ohm resistors connected to DNC pins have
been removed (TI uses them for internal testing only.) Pins 29 and 30 on
the AFE4400 pads appeared reversed, fixed that. Added single connectors
to utilize space better (compared to multiple pin connectors.)
Parts:
- removed C1: 0.1u, Capacitors_SMD:C_0603, symbol C
- removed P11: CONN_01X03, Wire_Pads:SolderWirePad_3x_0-8mmDrill, symbol CONN_01X03
- removed R1, R11, R12, R4, R7, R8: 130, Resistors_SMD:R_0603, symbol R
- added P11, P13, P14: CONN_01X01, Wire_Pads:SolderWirePad_single_0-8mmDrill, symbol CONN_01X01
- P10: footprint Morpheus_PPG_RevA:6_PADS_LED -> Crystals:crystal_FA238-TSX3225
Connections:
- wire segments 142 -> 141
- no-connect marks 9 -> 8
Other:
- moved on the sheet: C2, C3, P10, P9
